Commit message: setted up ros2 controller on gazebo simulation

File: description/robot.urdf.xacro (robot description, xacro)
@@ -2,14 +2,6 @@
 <robot xmlns:xacro="http://www.ros.org/wiki/xacro"  name="robot">
     <xacro:arg name="use_ros2_control" default="true"/>
-    <xacro:arg name="sim_mode" default="false"/>
+    <xacro:arg name="sim_mode" default="true"/>
     <xacro:include filename="robot_core.xacro" />
-    <!-- <xacro:if value="$(arg use_ros2_control)">
-        <xacro:include filename="ros2_control.xacro" />
-    </xacro:if>
-    <xacro:unless value="$(arg use_ros2_control)">
-        <xacro:include filename="gazebo_control.xacro" />
-    </xacro:unless> -->
-    <!-- <xacro:include filename="lidar.xacro" /> -->
-    <!-- <xacro:include filename="camera.xacro" /> -->
-    <!-- <xacro:include filename="depth_camera.xacro" /> -->
+    <xacro:include filename="ros2_control.xacro" />
 </robot>

File: description/robot_core.xacro (robot description, xacro)
@@ -5,5 +5,5 @@
     <xacro:property name="chassis_width" value="0.265"/>
     <xacro:property name="chassis_height" value="0.2"/>
-    <xacro:property name="chassis_mass" value="1.0"/>
+    <xacro:property name="chassis_mass" value="5"/>
     <xacro:property name="wheel_radius" value="0.05"/>
     <xacro:property name="wheel_thickness" value="0.026"/>
@@ -11,26 +11,18 @@
     <xacro:property name="rear_wheel_offset_x" value="0.3"/>
     <xacro:property name="rear_wheel_offset_y" value="0.2"/>
-    <xacro:property name="rear_wheel_offset_z" value="0.01"/>
-    <xacro:property name="front_wheel_offset_x" value="-0.2"/>
+    <xacro:property name="front_wheel_offset_x" value="0.1"/>
     <xacro:property name="front_wheel_offset_y" value="0.2"/>
-    <xacro:property name="front_wheel_offset_z" value="0.01"/>
     <xacro:property name="fork_length" value="0.25"/>
     <xacro:property name="fork_width" value="0.02"/>
     <xacro:property name="fork_thickness" value="0.02"/>
-    <xacro:property name="fork_mass" value="0.3"/>
+    <xacro:property name="fork_mass" value="0.01"/>
     <xacro:property name="fork_lift_mass" value="1.0"/>
     <xacro:property name="mast_height" value="0.5"/>
     <xacro:property name="mast_width" value="0.02"/>
-    <xacro:property name="mast_mass" value="0.3"/>
+    <xacro:property name="mast_mass" value="0.1"/>
     <xacro:property name="carriage_length" value="0.025"/>
     <xacro:property name="carriage_width" value="0.2"/>
     <xacro:property name="carriage_thickness" value="0.02"/>
-    <xacro:property name="carriage_mass" value="0.2"/>
-    <!-- derived sizes -->
-    <xacro:property name="cabin_x" value="${chassis_length/2}"/>
-    <xacro:property name="cabin_y" value="${chassis_width/2}"/>
-    <xacro:property name="cabin_z" value="${chassis_height*2}"/>
-    <xacro:property name="cabin_cx" value="${chassis_length/2}"/>
-    <xacro:property name="cabin_cz" value="${cabin_z/2}"/>
+    <xacro:property name="carriage_mass" value="0.1"/>
     <material name="white">
         <color rgba="1 1 1 1" />
@@ -63,5 +55,5 @@
         <parent link="base_link"/>
         <child link="chassis"/>
-        <origin xyz="${-rear_wheel_offset_x} 0 ${-rear_wheel_offset_z}"/>
+        <origin xyz="${-rear_wheel_offset_x} 0 ${wheel_radius}"/>
     </joint>
     <link name="chassis">
@@ -87,5 +79,5 @@
     </gazebo>
     <!-- CABIN LINK -->
-    <joint name="cabin_joint" type="fixed">
+    <!-- <joint name="cabin_joint" type="fixed">
         <parent link="base_link"/>
         <child link="cabin"/>
@@ -106,14 +98,58 @@
             </geometry>
         </collision>
-        <!-- inertial: place COM at geometric center of the cabin box -->
+ì
         <xacro:inertial_box mass="0.5" x="${cabin_x}" y="${cabin_y}" z="${cabin_z}">
             <origin xyz="${cabin_cx} 0 ${cabin_cz}" rpy="0 0 0"/>
         </xacro:inertial_box>
+    </link> -->
+    <!-- RIGHT REAR STEERING JOINT -->
+    <joint name="right_rear_steer_joint" type="revolute">
+        <parent link="chassis"/>
+        <child link="right_rear_wheel_steer"/>
+        <origin xyz="${rear_wheel_offset_x} ${rear_wheel_offset_y} 0" rpy="0 0 0"/>
+        <axis xyz="0 0 1"/>
+        <limit lower="-0.5" upper="0.5" effort="5.0" velocity="1.0"/>
+    </joint>
+    <link name="right_rear_wheel_steer">
+        <visual>
+            <geometry><box size="0.01 0.01 0.01"/></geometry> <!-- dummy link -->
+        </visual>
+        <collision>
+            <geometry><box size="0.01 0.01 0.01"/></geometry>
+        </collision>
+        <inertial>
+            <mass value="0.01"/>
+            <origin xyz="0 0 0" rpy="0 0 0"/>
+            <inertia ixx="0.0001" ixy="0" ixz="0" iyy="0.0001" iyz="0" izz="0.0001"/>
+        </inertial>
+    </link>
+    <!-- RIGHT REAR WHEEL -->
+    <joint name="right_rear_wheel_joint" type="continuous">
+        <parent link="right_rear_wheel_steer"/>
+        <child link="right_rear_wheel"/>
+        <origin xyz="0 0 0" rpy="-${pi/2} 0 0"/>
+        <axis xyz="0 0 1"/>
+    </joint>
+    <link name="right_rear_wheel">
+        <visual>
+            <geometry>
+                <cylinder radius="${wheel_radius}" length="${wheel_thickness}"/>
+            </geometry>
+            <material name="blue"/>
+        </visual>
+        <collision>
+            <geometry>
+                <cylinder radius="${wheel_radius}" length="${wheel_thickness}"/>
+            </geometry>
+        </collision>
+        <xacro:inertial_cylinder mass="${wheel_mass}" length="${wheel_thickness}" radius="${wheel_radius}">
+            <origin xyz="0 0 0" rpy="0 0 0"/>
+        </xacro:inertial_cylinder>
     </link>
     <!-- LEFT REAR STEERING JOINT -->
     <joint name="left_rear_steer_joint" type="revolute">
-        <parent link="base_link"/>
+        <parent link="chassis"/>
         <child link="left_rear_wheel_steer"/>
-        <origin xyz="0 ${rear_wheel_offset_y} 0" rpy="0 0 0"/>
+        <origin xyz="${rear_wheel_offset_x} ${-rear_wheel_offset_y} 0" rpy="0 0 0"/>
         <axis xyz="0 0 1"/>
         <limit lower="-0.5" upper="0.5" effort="5.0" velocity="1.0"/>
@@ -123,49 +159,21 @@
             <geometry><box size="0.01 0.01 0.01"/></geometry> <!-- dummy link -->
         </visual>
-    </link>
-    <!-- LEFT REAR WHEEL -->
+        <collision>
+            <geometry><box size="0.01 0.01 0.01"/></geometry>
+        </collision>
+        <inertial>
+            <mass value="0.01"/>
+            <origin xyz="0 0 0" rpy="0 0 0"/>
+            <inertia ixx="0.0001" ixy="0" ixz="0" iyy="0.0001" iyz="0" izz="0.0001"/>
+        </inertial>
+    </link>
+    <!-- LEFT REAR WHEEL LINK -->
     <joint name="left_rear_wheel_joint" type="continuous">
         <parent link="left_rear_wheel_steer"/>
         <child link="left_rear_wheel"/>
-        <origin xyz="0 0 0" rpy="-${pi/2} 0 0"/>
-        <axis xyz="0 0 1"/>
-    </joint>
-    <link name="left_rear_wheel">
-        <visual>
-            <geometry>
-                <cylinder radius="${wheel_radius}" length="${wheel_thickness}"/>
-            </geometry>
-            <material name="blue"/>
-        </visual>
-        <collision>
-            <geometry>
-                <cylinder radius="${wheel_radius}" length="${wheel_thickness}"/>
-            </geometry>
-        </collision>
-        <xacro:inertial_cylinder mass="${wheel_mass}" length="${wheel_thickness}" radius="${wheel_radius}">
-            <origin xyz="0 0 0" rpy="0 0 0"/>
-        </xacro:inertial_cylinder>
-    </link>
-    <!-- RIGHT REAR STEERING JOINT -->
-    <joint name="right_rear_steer_joint" type="revolute">
-        <parent link="base_link"/>
-        <child link="right_rear_wheel_steer"/>
-        <origin xyz="0 ${-rear_wheel_offset_y} 0" rpy="0 0 0"/>
-        <axis xyz="0 0 1"/>
-        <limit lower="-0.5" upper="0.5" effort="5.0" velocity="1.0"/>
-    </joint>
-    <link name="right_rear_wheel_steer">
-        <visual>
-            <geometry><box size="0.01 0.01 0.01"/></geometry> <!-- dummy link -->
-        </visual>
-    </link>
-    <!-- RIGHT REAR WHEEL LINK -->
-    <joint name="right_rear_wheel_joint" type="continuous">
-        <parent link="right_rear_wheel_steer"/>
-        <child link="right_rear_wheel"/>
         <origin xyz="0 0 0" rpy="${pi/2} 0 0" />
         <axis xyz="0 0 -1"/>
     </joint>
-    <link name="right_rear_wheel">
+    <link name="left_rear_wheel">
         <visual>
             <geometry>
@@ -183,15 +191,15 @@
         </xacro:inertial_cylinder>
     </link>
-    <gazebo reference="right_rear_wheel">
+    <gazebo reference="left_rear_wheel">
         <material>Gazebo/Blue</material>
     </gazebo>
-    <!-- LEFT FRONT WHEEL LINK -->
-    <joint name="left_front_wheel_joint" type="continuous">
-        <parent link="base_link"/>
-        <child link="left_front_wheel"/>
+    <!-- right FRONT WHEEL LINK -->
+    <joint name="right_front_wheel_joint" type="continuous">
+        <parent link="chassis"/>
+        <child link="right_front_wheel"/>
         <origin xyz="${front_wheel_offset_x} ${front_wheel_offset_y} 0" rpy="-${pi/2} 0 0" />
         <axis xyz="0 0 1"/>
     </joint>
-    <link name="left_front_wheel">
+    <link name="right_front_wheel">
         <visual>
             <geometry>
@@ -209,15 +217,15 @@
         </xacro:inertial_cylinder>
     </link>
-    <gazebo reference="left_front_wheel">
+    <gazebo reference="right_front_wheel">
         <material>Gazebo/Blue</material>
     </gazebo>
-    <!-- RIGHT FRONT WHEEL LINK -->
-    <joint name="right_front_wheel_joint" type="continuous">
-        <parent link="base_link"/>
-        <child link="right_front_wheel"/>
+    <!-- left FRONT WHEEL LINK -->
+    <joint name="left_front_wheel_joint" type="continuous">
+        <parent link="chassis"/>
+        <child link="left_front_wheel"/>
         <origin xyz="${front_wheel_offset_x} ${-front_wheel_offset_y} 0" rpy="${pi/2} 0 0" />
         <axis xyz="0 0 -1"/>
     </joint>
-    <link name="right_front_wheel">
+    <link name="left_front_wheel">
         <visual>
             <geometry>
@@ -235,5 +243,5 @@
         </xacro:inertial_cylinder>
     </link>
-    <gazebo reference="right_front_wheel">
+    <gazebo reference="left_front_wheel">
         <material>Gazebo/Blue</material>
     </gazebo>
@@ -284,5 +292,27 @@
         <limit lower="0" upper="${mast_height}" effort="10" velocity="0.1"/>
     </joint>
-    <!-- LEFT FORK -->
+    <!-- right FORK -->
+    <link name="fork_right">
+        <visual>
+            <geometry>
+                <box size="${fork_length} ${fork_width} ${fork_thickness}"/>
+            </geometry>
+            <material name="black"/>
+        </visual>
+        <collision>
+            <geometry>
+                <box size="${fork_length} ${fork_width} ${fork_thickness}"/>
+            </geometry>
+        </collision>
+        <xacro:inertial_box mass="${fork_mass}" x="${fork_length}" y="${fork_width}" z="${fork_thickness}">
+        <origin xyz="${fork_length/2} 0 0"/>
+        </xacro:inertial_box>
+    </link>
+    <joint name="fork_right_joint" type="fixed">
+        <parent link="fork_carriage"/>
+        <child link="fork_right"/>
+        <origin xyz="${-fork_length/2+carriage_length/2} ${(carriage_width/2+fork_width)} 0" rpy="0 0 ${pi}"/>
+    </joint>
+    <!-- left FORK -->
     <link name="fork_left">
         <visual>
@@ -304,26 +334,4 @@
         <parent link="fork_carriage"/>
         <child link="fork_left"/>
-        <origin xyz="${-fork_length/2+carriage_length/2} ${(carriage_width/2+fork_width)} 0" rpy="0 0 ${pi}"/>
-    </joint>
-    <!-- RIGHT FORK -->
-    <link name="fork_right">
-        <visual>
-            <geometry>
-                <box size="${fork_length} ${fork_width} ${fork_thickness}"/>
-            </geometry>
-            <material name="black"/>
-        </visual>
-        <collision>
-            <geometry>
-                <box size="${fork_length} ${fork_width} ${fork_thickness}"/>
-            </geometry>
-        </collision>
-        <xacro:inertial_box mass="${fork_mass}" x="${fork_length}" y="${fork_width}" z="${fork_thickness}">
-        <origin xyz="${fork_length/2} 0 0"/>
-        </xacro:inertial_box>
-    </link>
-    <joint name="fork_right_joint" type="fixed">
-        <parent link="fork_carriage"/>
-        <child link="fork_right"/>
         <origin xyz="${-fork_length/2+carriage_length/2} ${-(carriage_width/2+fork_width)} 0" rpy="0 0 ${pi}"/>
     </joint>

File: description/ros2_control.xacro (robot description, xacro)
@@ -1,61 +1,43 @@
 <?xml version="1.0"?>
 <robot xmlns:xacro="http://www.ros.org/wiki/xacro">
-    <xacro:unless value="$(arg sim_mode)">
-        <ros2_control name="RealRobot" type="system">
-            <hardware>
-                <plugin>diffdrive_arduino/DiffDriveArduino</plugin>
-                <param name="left_wheel_name">left_wheel_joint</param>
-                <param name="right_wheel_name">right_wheel_joint</param>
-                <param name="loop_rate">30</param>
-                <param name="device">/dev/ttyUSB0</param>
-                <param name="baud_rate">57600</param>
-                <param name="timeout">1000</param>
-                <param name="enc_counts_per_rev">3436</param>
-            </hardware>
-            <joint name="left_wheel_joint">
-                <command_interface name="velocity">
-                    <param name="min">-10</param>
-                    <param name="max">10</param>
-                </command_interface>
-                <state_interface name="velocity"/>
-                <state_interface name="position"/>
-            </joint>
-            <joint name="right_wheel_joint">
-                <command_interface name="velocity">
-                    <param name="min">-10</param>
-                    <param name="max">10</param>
-                </command_interface>
-                <state_interface name="velocity"/>
-                <state_interface name="position"/>
-            </joint>
-        </ros2_control>
-    </xacro:unless>
-    <xacro:if value="$(arg sim_mode)">
-        <ros2_control name="GazeboSystem" type="system">
-            <hardware>
-                <plugin>gazebo_ros2_control/GazeboSystem</plugin>
-            </hardware>
-            <joint name="left_wheel_joint">
-                <command_interface name="velocity">
-                    <param name="min">-10</param>
-                    <param name="max">10</param>
-                </command_interface>
-                <state_interface name="velocity"/>
-                <state_interface name="position"/>
-            </joint>
-            <joint name="right_wheel_joint">
-                <command_interface name="velocity">
-                    <param name="min">-10</param>
-                    <param name="max">10</param>
-                </command_interface>
-                <state_interface name="velocity"/>
-                <state_interface name="position"/>
-            </joint>
-        </ros2_control>
-    </xacro:if>
+   <!-- Hardware interface for the simulated environment -->
+    <ros2_control name="GazeboSystem" type="system">
+        <hardware>
+            <plugin>gz_ros2_control/GazeboSimSystem</plugin>
+        </hardware>
+        <joint name="left_front_wheel_joint">
+            <command_interface name="velocity"/>
+            <state_interface name="position"/>
+            <state_interface name="velocity"/>
+        </joint>
+        <joint name="right_front_wheel_joint">
+            <command_interface name="velocity"/>
+            <state_interface name="position"/>
+            <state_interface name="velocity"/>
+        </joint>
+        <joint name="left_rear_wheel_joint">
+            <state_interface name="position"/>
+            <state_interface name="velocity"/>
+        </joint>
+        <joint name="right_rear_wheel_joint">
+            <state_interface name="position"/>
+            <state_interface name="velocity"/>
+        </joint>
+        <joint name="right_rear_steer_joint">
+            <command_interface name="position"/>
+            <state_interface name="position"/>
+        </joint>
+        <joint name="left_rear_steer_joint">
+            <command_interface name="position"/>
+            <state_interface name="position"/>
+        </joint>
+        <joint name="fork_carriage_joint">
+            <command_interface name="position"/>
+            <state_interface name="position"/>
+        </joint>
+    </ros2_control>
     <gazebo>
-        <plugin name="gazebo_ros2_control" filename="libgazebo_ros2_control.so">
-            <parameters>$(find forklift_one)/config/my_controllers.yaml</parameters>
-            <parameters>$(find forklift_one)/config/gaz_ros2_ctl_use_sim.yaml</parameters>
+        <plugin name="gz_ros2_control::GazeboSimROS2ControlPlugin" filename="libgz_ros2_control-system.so">
+        <parameters>$(find forklift_one)/config/forklift_controllers.yaml</parameters>
         </plugin>
     </gazebo>
