Commit message: Added driving controller in the simulation

File: description/robot_core.xacro (robot description, xacro)
@@ -4,5 +4,5 @@
     <xacro:property name="chassis_length" value="0.4"/>
     <xacro:property name="chassis_width" value="0.265"/>
-    <xacro:property name="chassis_height" value="0.2"/>
+    <xacro:property name="chassis_height" value="0.15"/>
     <xacro:property name="chassis_mass" value="5"/>
     <xacro:property name="wheel_radius" value="0.05"/>
@@ -79,28 +79,26 @@
     </gazebo>
     <!-- CABIN LINK -->
-    <!-- <joint name="cabin_joint" type="fixed">
-        <parent link="base_link"/>
+    <joint name="cabin_joint" type="fixed">
+        <parent link="chassis"/>
         <child link="cabin"/>
-        <origin xyz="${-rear_wheel_offset_x} 0 ${-rear_wheel_offset_z}"/>
+        <origin xyz="0 0 0"/>
     </joint>
     <link name="cabin">
         <visual>
-            <origin xyz="${cabin_cx} 0 ${cabin_cz}" rpy="0 0 0"/>
-            <geometry>
-                <box size="${cabin_x} ${cabin_y} ${cabin_z}"/>
+            <origin xyz="${chassis_length*0.6} 0 ${chassis_height*1.5}" rpy="0 0 0"/>
+            <geometry>
+                <box size="${chassis_length/2} ${chassis_width/2} ${chassis_height*2}"/>
             </geometry>
             <material name="orange"/>
         </visual>
         <collision>
-            <origin xyz="${cabin_cx} 0 ${cabin_cz}" rpy="0 0 0"/>
-            <geometry>
-                <box size="${cabin_x} ${cabin_y} ${cabin_z}"/>
-            </geometry>
-        </collision>
-ì
-        <xacro:inertial_box mass="0.5" x="${cabin_x}" y="${cabin_y}" z="${cabin_z}">
-            <origin xyz="${cabin_cx} 0 ${cabin_cz}" rpy="0 0 0"/>
-        </xacro:inertial_box>
-    </link> -->
+            <geometry>
+                <box size="${chassis_length/2} ${chassis_width/2} ${chassis_height*2}"/>
+            </geometry>
+        </collision>
+        <xacro:inertial_box mass="1.0" x="${chassis_length/2}" y="${chassis_width/2}" z="${chassis_height*2}">
+            <origin xyz="${chassis_length*0.6} 0 ${chassis_height*1.5}" rpy="0 0 0"/>
+        </xacro:inertial_box>
+    </link>
     <!-- RIGHT REAR STEERING JOINT -->
     <joint name="right_rear_steer_joint" type="revolute">

File: description/ros2_control.xacro (robot description, xacro)
@@ -6,4 +6,5 @@
             <plugin>gz_ros2_control/GazeboSimSystem</plugin>
         </hardware>
+        <!-- Front wheels (driving) -->
         <joint name="left_front_wheel_joint">
             <command_interface name="velocity"/>
@@ -16,23 +17,31 @@
             <state_interface name="velocity"/>
         </joint>
+        <!-- Rear wheels (driven by chassis if fixed, but normally they rotate) -->
         <joint name="left_rear_wheel_joint">
+            <command_interface name="velocity"/>
             <state_interface name="position"/>
             <state_interface name="velocity"/>
         </joint>
         <joint name="right_rear_wheel_joint">
+            <command_interface name="velocity"/>
             <state_interface name="position"/>
             <state_interface name="velocity"/>
         </joint>
+        <!-- Steering joints -->
         <joint name="right_rear_steer_joint">
             <command_interface name="position"/>
             <state_interface name="position"/>
+            <state_interface name="velocity"/>
         </joint>
         <joint name="left_rear_steer_joint">
             <command_interface name="position"/>
             <state_interface name="position"/>
+            <state_interface name="velocity"/>
         </joint>
+        <!-- Lift mechanism -->
         <joint name="fork_carriage_joint">
             <command_interface name="position"/>
             <state_interface name="position"/>
+            <state_interface name="velocity"/>
         </joint>
     </ros2_control>

Commit message: fix: changed joint type for caster wheels, should have been revolute, not continuous

File: description/robot_core.xacro (robot description, xacro)
@@ -2,12 +2,12 @@
 <robot xmlns:xacro="http://www.ros.org/wiki/xacro" >
     <xacro:include filename="inertial_macros.xacro"/>
-    <xacro:property name="chassis_length" value="0.4"/>
+    <xacro:property name="chassis_length" value="0.6"/>
     <xacro:property name="chassis_width" value="0.265"/>
     <xacro:property name="chassis_height" value="0.15"/>
     <xacro:property name="chassis_mass" value="5"/>
-    <xacro:property name="wheel_radius" value="0.05"/>
+    <xacro:property name="wheel_radius" value="0.1"/>
     <xacro:property name="wheel_thickness" value="0.026"/>
     <xacro:property name="wheel_mass" value="0.05"/>
-    <xacro:property name="rear_wheel_offset_x" value="0.3"/>
+    <xacro:property name="rear_wheel_offset_x" value="0.5"/>
     <xacro:property name="rear_wheel_offset_y" value="0.2"/>
     <xacro:property name="front_wheel_offset_x" value="0.1"/>
@@ -93,4 +93,5 @@
         </visual>
         <collision>
+            <origin xyz="${chassis_length*0.6} 0 ${chassis_height*1.5}" rpy="0 0 0"/>
             <geometry>
                 <box size="${chassis_length/2} ${chassis_width/2} ${chassis_height*2}"/>
@@ -123,9 +124,11 @@
     </link>
     <!-- RIGHT REAR WHEEL -->
-    <joint name="right_rear_wheel_joint" type="continuous">
+    <joint name="right_rear_wheel_joint" type="revolute">
         <parent link="right_rear_wheel_steer"/>
         <child link="right_rear_wheel"/>
         <origin xyz="0 0 0" rpy="-${pi/2} 0 0"/>
         <axis xyz="0 0 1"/>
+        <limit lower="-1000" upper="1000" effort="0.0" velocity="1000"/> <!-- essentially free rotation -->
+        <dynamics damping="0.05" friction="0.0"/> <!-- small damping to stabilize -->
     </joint>
     <link name="right_rear_wheel">
@@ -140,4 +143,14 @@
                 <cylinder radius="${wheel_radius}" length="${wheel_thickness}"/>
             </geometry>
+            <surface>
+                <friction>
+                    <ode>
+                        <mu>5.0</mu>       <!-- longitudinal friction -->
+                        <mu2>5.0</mu2>     <!-- lateral friction -->
+                        <slip1>0.0</slip1>
+                        <slip2>0.0</slip2>
+                    </ode>
+                </friction>
+            </surface>
         </collision>
         <xacro:inertial_cylinder mass="${wheel_mass}" length="${wheel_thickness}" radius="${wheel_radius}">
@@ -167,9 +180,11 @@
     </link>
     <!-- LEFT REAR WHEEL LINK -->
-    <joint name="left_rear_wheel_joint" type="continuous">
+    <joint name="left_rear_wheel_joint" type="revolute">
         <parent link="left_rear_wheel_steer"/>
         <child link="left_rear_wheel"/>
         <origin xyz="0 0 0" rpy="${pi/2} 0 0" />
         <axis xyz="0 0 -1"/>
+        <limit lower="-1000" upper="1000" effort="0.0" velocity="1000"/> <!-- essentially free rotation -->
+        <dynamics damping="0.05" friction="0.0"/> <!-- small damping to stabilize -->
     </joint>
     <link name="left_rear_wheel">
@@ -182,6 +197,16 @@
         <collision>
             <geometry>
-                <sphere radius="${wheel_radius}"/>
-            </geometry>
+                <cylinder radius="${wheel_radius}" length="${wheel_thickness}"/>
+            </geometry>
+            <surface>
+                <friction>
+                    <ode>
+                        <mu>5.0</mu>       <!-- longitudinal friction -->
+                        <mu2>5.0</mu2>     <!-- lateral friction -->
+                        <slip1>0.0</slip1>
+                        <slip2>0.0</slip2>
+                    </ode>
+                </friction>
+            </surface>
         </collision>
         <xacro:inertial_cylinder mass="${wheel_mass}" length="${wheel_thickness}" radius="${wheel_radius}">
@@ -208,6 +233,14 @@
         <collision>
             <geometry>
-                <sphere radius="${wheel_radius}"/>
-            </geometry>
+                <cylinder radius="${wheel_radius}" length="${wheel_thickness}"/>
+            </geometry>
+            <!-- <surface>
+                <friction>
+                    <ode>
+                        <mu>0.01</mu>
+                        <mu2>0.1</mu2>
+                    </ode>
+                </friction>
+            </surface> -->
         </collision>
         <xacro:inertial_cylinder mass="${wheel_mass}" length="${wheel_thickness}" radius="${wheel_radius}">
@@ -234,6 +267,14 @@
         <collision>
             <geometry>
-                <sphere radius="${wheel_radius}"/>
-            </geometry>
+                <cylinder radius="${wheel_radius}" length="${wheel_thickness}"/>
+            </geometry>
+            <!-- <surface>
+                <friction>
+                    <ode>
+                        <mu>0.01</mu>
+                        <mu2>0.1</mu2>
+                    </ode>
+                </friction>
+            </surface> -->
         </collision>
         <xacro:inertial_cylinder mass="${wheel_mass}" length="${wheel_thickness}" radius="${wheel_radius}">
@@ -264,5 +305,5 @@
         <parent link="chassis"/>
         <child link="mast"/>
-        <origin xyz="${-mast_width/2} 0 ${mast_height/2}" rpy="0 0 0"/>
+        <origin xyz="${-mast_width/2} 0 ${wheel_radius*0.1+chassis_height}" rpy="0 0 0"/>
     </joint>
     <!-- FORK CARRIAGE -->

Commit message: fix: adjusted axis orientation

File: description/robot_core.xacro (robot description, xacro)
@@ -222,5 +222,5 @@
         <child link="right_front_wheel"/>
         <origin xyz="${front_wheel_offset_x} ${front_wheel_offset_y} 0" rpy="-${pi/2} 0 0" />
-        <axis xyz="0 0 1"/>
+        <axis xyz="0 0 -1"/>
     </joint>
     <link name="right_front_wheel">
@@ -256,5 +256,5 @@
         <child link="left_front_wheel"/>
         <origin xyz="${front_wheel_offset_x} ${-front_wheel_offset_y} 0" rpy="${pi/2} 0 0" />
-        <axis xyz="0 0 -1"/>
+        <axis xyz="0 0 1"/>
     </joint>
     <link name="left_front_wheel">

Commit message: fix: changed steering axis orientation

File: description/robot_core.xacro (robot description, xacro)
@@ -107,5 +107,5 @@
         <child link="right_rear_wheel_steer"/>
         <origin xyz="${rear_wheel_offset_x} ${rear_wheel_offset_y} 0" rpy="0 0 0"/>
-        <axis xyz="0 0 1"/>
+        <axis xyz="0 0 -1"/>
         <limit lower="-0.5" upper="0.5" effort="5.0" velocity="1.0"/>
     </joint>
@@ -163,5 +163,5 @@
         <child link="left_rear_wheel_steer"/>
         <origin xyz="${rear_wheel_offset_x} ${-rear_wheel_offset_y} 0" rpy="0 0 0"/>
-        <axis xyz="0 0 1"/>
+        <axis xyz="0 0 -1"/>
         <limit lower="-0.5" upper="0.5" effort="5.0" velocity="1.0"/>
     </joint>

Commit message: Changed the urdf to match geometry of real robot

File: description/robot_core.xacro (robot description, xacro)
@@ -2,26 +2,27 @@
 <robot xmlns:xacro="http://www.ros.org/wiki/xacro" >
     <xacro:include filename="inertial_macros.xacro"/>
-    <xacro:property name="chassis_length" value="0.6"/>
-    <xacro:property name="chassis_width" value="0.265"/>
-    <xacro:property name="chassis_height" value="0.15"/>
+    <xacro:property name="chassis_length" value="0.215"/>
+    <xacro:property name="chassis_width" value="0.09"/>
+    <xacro:property name="chassis_height" value="0.005"/>
     <xacro:property name="chassis_mass" value="5"/>
-    <xacro:property name="wheel_radius" value="0.1"/>
-    <xacro:property name="wheel_thickness" value="0.026"/>
+    <xacro:property name="front_wheel_radius" value="0.0425"/>
+    <xacro:property name="rear_wheel_radius" value="0.0375"/>
+    <xacro:property name="wheel_thickness" value="0.025"/>
     <xacro:property name="wheel_mass" value="0.05"/>
-    <xacro:property name="rear_wheel_offset_x" value="0.5"/>
-    <xacro:property name="rear_wheel_offset_y" value="0.2"/>
-    <xacro:property name="front_wheel_offset_x" value="0.1"/>
-    <xacro:property name="front_wheel_offset_y" value="0.2"/>
-    <xacro:property name="fork_length" value="0.25"/>
-    <xacro:property name="fork_width" value="0.02"/>
-    <xacro:property name="fork_thickness" value="0.02"/>
+    <xacro:property name="rear_wheel_offset_x" value="0.215"/>
+    <xacro:property name="rear_wheel_offset_y" value="0.075"/>
+    <xacro:property name="front_wheel_offset_x" value="0.0"/>
+    <xacro:property name="front_wheel_offset_y" value="0.07"/>
+    <xacro:property name="mast_offset_x" value="0.07"/>
+    <xacro:property name="mast_height" value="0.170"/>
+    <xacro:property name="mast_width" value="0.01"/>
+    <xacro:property name="mast_mass" value="0.1"/>
+    <xacro:property name="fork_length" value="0.1"/>
+    <xacro:property name="fork_width" value="0.01"/>
+    <xacro:property name="fork_thickness" value="0.01"/>
     <xacro:property name="fork_mass" value="0.01"/>
-    <xacro:property name="fork_lift_mass" value="1.0"/>
-    <xacro:property name="mast_height" value="0.5"/>
-    <xacro:property name="mast_width" value="0.02"/>
-    <xacro:property name="mast_mass" value="0.1"/>
-    <xacro:property name="carriage_length" value="0.025"/>
-    <xacro:property name="carriage_width" value="0.2"/>
-    <xacro:property name="carriage_thickness" value="0.02"/>
+    <xacro:property name="carriage_length" value="0.01"/>
+    <xacro:property name="carriage_width" value="0.140"/>
+    <xacro:property name="carriage_thickness" value="0.01"/>
     <xacro:property name="carriage_mass" value="0.1"/>
     <material name="white">
@@ -55,5 +56,5 @@
         <parent link="base_link"/>
         <child link="chassis"/>
-        <origin xyz="${-rear_wheel_offset_x} 0 ${wheel_radius}"/>
+        <origin xyz="${-rear_wheel_offset_x} 0 ${front_wheel_radius}"/>
     </joint>
     <link name="chassis">
@@ -78,28 +79,4 @@
         <material>Gazebo/Orange</material>
     </gazebo>
-    <!-- CABIN LINK -->
-    <joint name="cabin_joint" type="fixed">
-        <parent link="chassis"/>
-        <child link="cabin"/>
-        <origin xyz="0 0 0"/>
-    </joint>
-    <link name="cabin">
-        <visual>
-            <origin xyz="${chassis_length*0.6} 0 ${chassis_height*1.5}" rpy="0 0 0"/>
-            <geometry>
-                <box size="${chassis_length/2} ${chassis_width/2} ${chassis_height*2}"/>
-            </geometry>
-            <material name="orange"/>
-        </visual>
-        <collision>
-            <origin xyz="${chassis_length*0.6} 0 ${chassis_height*1.5}" rpy="0 0 0"/>
-            <geometry>
-                <box size="${chassis_length/2} ${chassis_width/2} ${chassis_height*2}"/>
-            </geometry>
-        </collision>
-        <xacro:inertial_box mass="1.0" x="${chassis_length/2}" y="${chassis_width/2}" z="${chassis_height*2}">
-            <origin xyz="${chassis_length*0.6} 0 ${chassis_height*1.5}" rpy="0 0 0"/>
-        </xacro:inertial_box>
-    </link>
     <!-- RIGHT REAR STEERING JOINT -->
     <joint name="right_rear_steer_joint" type="revolute">
@@ -135,17 +112,17 @@
         <visual>
             <geometry>
-                <cylinder radius="${wheel_radius}" length="${wheel_thickness}"/>
-            </geometry>
-            <material name="blue"/>
-        </visual>
-        <collision>
-            <geometry>
-                <cylinder radius="${wheel_radius}" length="${wheel_thickness}"/>
+                <cylinder radius="${front_wheel_radius}" length="${wheel_thickness}"/>
+            </geometry>
+            <material name="blue"/>
+        </visual>
+        <collision>
+            <geometry>
+                <cylinder radius="${rear_wheel_radius}" length="${wheel_thickness}"/>
             </geometry>
             <surface>
                 <friction>
                     <ode>
-                        <mu>5.0</mu>       <!-- longitudinal friction -->
-                        <mu2>5.0</mu2>     <!-- lateral friction -->
+                        <mu>1.0</mu>       <!-- longitudinal friction -->
+                        <mu2>1.0</mu2>     <!-- lateral friction -->
                         <slip1>0.0</slip1>
                         <slip2>0.0</slip2>
@@ -154,5 +131,5 @@
             </surface>
         </collision>
-        <xacro:inertial_cylinder mass="${wheel_mass}" length="${wheel_thickness}" radius="${wheel_radius}">
+        <xacro:inertial_cylinder mass="${wheel_mass}" length="${wheel_thickness}" radius="${rear_wheel_radius}">
             <origin xyz="0 0 0" rpy="0 0 0"/>
         </xacro:inertial_cylinder>
@@ -191,17 +168,17 @@
         <visual>
             <geometry>
-                <cylinder radius="${wheel_radius}" length="${wheel_thickness}"/>
-            </geometry>
-            <material name="blue"/>
-        </visual>
-        <collision>
-            <geometry>
-                <cylinder radius="${wheel_radius}" length="${wheel_thickness}"/>
+                <cylinder radius="${rear_wheel_radius}" length="${wheel_thickness}"/>
+            </geometry>
+            <material name="blue"/>
+        </visual>
+        <collision>
+            <geometry>
+                <cylinder radius="${rear_wheel_radius}" length="${wheel_thickness}"/>
             </geometry>
             <surface>
                 <friction>
                     <ode>
-                        <mu>5.0</mu>       <!-- longitudinal friction -->
-                        <mu2>5.0</mu2>     <!-- lateral friction -->
+                        <mu>1.0</mu>       <!-- longitudinal friction -->
+                        <mu2>1.0</mu2>     <!-- lateral friction -->
                         <slip1>0.0</slip1>
                         <slip2>0.0</slip2>
@@ -210,5 +187,5 @@
             </surface>
         </collision>
-        <xacro:inertial_cylinder mass="${wheel_mass}" length="${wheel_thickness}" radius="${wheel_radius}">
+        <xacro:inertial_cylinder mass="${wheel_mass}" length="${wheel_thickness}" radius="${rear_wheel_radius}">
             <origin xyz="0 0 0" rpy="0 0 0"/>
         </xacro:inertial_cylinder>
@@ -227,11 +204,11 @@
         <visual>
             <geometry>
-                <cylinder radius="${wheel_radius}" length="${wheel_thickness}"/>
-            </geometry>
-            <material name="blue"/>
-        </visual>
-        <collision>
-            <geometry>
-                <cylinder radius="${wheel_radius}" length="${wheel_thickness}"/>
+                <cylinder radius="${front_wheel_radius}" length="${wheel_thickness}"/>
+            </geometry>
+            <material name="blue"/>
+        </visual>
+        <collision>
+            <geometry>
+                <cylinder radius="${front_wheel_radius}" length="${wheel_thickness}"/>
             </geometry>
             <!-- <surface>
@@ -244,5 +221,5 @@
             </surface> -->
         </collision>
-        <xacro:inertial_cylinder mass="${wheel_mass}" length="${wheel_thickness}" radius="${wheel_radius}">
+        <xacro:inertial_cylinder mass="${wheel_mass}" length="${wheel_thickness}" radius="${front_wheel_radius}">
             <origin xyz="0 0 0" rpy="0 0 0"/>
         </xacro:inertial_cylinder>
@@ -261,11 +238,11 @@
         <visual>
             <geometry>
-                <cylinder radius="${wheel_radius}" length="${wheel_thickness}"/>
-            </geometry>
-            <material name="blue"/>
-        </visual>
-        <collision>
-            <geometry>
-                <cylinder radius="${wheel_radius}" length="${wheel_thickness}"/>
+                <cylinder radius="${front_wheel_radius}" length="${wheel_thickness}"/>
+            </geometry>
+            <material name="blue"/>
+        </visual>
+        <collision>
+            <geometry>
+                <cylinder radius="${front_wheel_radius}" length="${wheel_thickness}"/>
             </geometry>
             <!-- <surface>
@@ -278,5 +255,5 @@
             </surface> -->
         </collision>
-        <xacro:inertial_cylinder mass="${wheel_mass}" length="${wheel_thickness}" radius="${wheel_radius}">
+        <xacro:inertial_cylinder mass="${wheel_mass}" length="${wheel_thickness}" radius="${front_wheel_radius}">
             <origin xyz="0 0 0" rpy="0 0 0"/>
         </xacro:inertial_cylinder>
@@ -299,5 +276,5 @@
         </collision>
         <xacro:inertial_box mass="${mast_mass}" x="${mast_width}" y="${mast_width}" z="${mast_height}">
-            <origin xyz="${mast_width/2} 0 ${mast_height/2}" rpy="0 0 0"/>
+            <origin xyz="${mast_width/2} 0 ${mast_height/2+0.01}" rpy="0 0 0"/>
         </xacro:inertial_box>
     </link>
@@ -305,5 +282,5 @@
         <parent link="chassis"/>
         <child link="mast"/>
-        <origin xyz="${-mast_width/2} 0 ${wheel_radius*0.1+chassis_height}" rpy="0 0 0"/>
+        <origin xyz="${-mast_offset_x+mast_width/2} 0 ${-front_wheel_radius+mast_height/2}" rpy="0 0 0"/>
     </joint>
     <!-- FORK CARRIAGE -->

Commit message: fix: corrected typos and updated readme

File: description/robot_core.xacro (robot description, xacro)
@@ -112,5 +112,5 @@
         <visual>
             <geometry>
-                <cylinder radius="${front_wheel_radius}" length="${wheel_thickness}"/>
+                <cylinder radius="${rear_wheel_radius}" length="${wheel_thickness}"/>
             </geometry>
             <material name="blue"/>
